Commit message: Circle detection problem - using Opencv3 instead of Opencv2

File: src/scara_cpe_4students/scara_cpe_description/urdf/scara_cpe.xacro (robot description, xacro)
@@ -44,9 +44,9 @@
     <inertial>
       <origin xyz="0 0.04 0" rpy="0 0 0" />
-      <mass value="0.1"/>
-      <inertia
-        ixx="0.00003" ixy="1e-12" ixz="1e-12"
-        iyy="0.00003" iyz="1e-12"
-        izz="0.00003"/>
+      <mass value="0.0001"/>
+     <inertia
+        ixx="0.0001" ixy="1e-12" ixz="1e-12"
+        iyy="0.0001" iyz="1e-12"
+        izz="0.0001"/>
     </inertial>
   </link>
@@ -66,5 +66,5 @@
     <inertial>
       <origin xyz="0 0.02 0" rpy="0 0 0" />
-      <mass value="0.1"/>
+      <mass value="0.0001"/>
       <inertia
         ixx="0.0001" ixy="1e-12" ixz="1e-12"
